File: ASTRA_Base_Station.kicad_sch (KiCad schematic)
At the start: 24 parts, among them J1 LSS Conn, J2 24V, J3 24V, J4 24V, J5 5V, U2 Adafruit FeatherWing, U3 NEOM9N, U4 BNO055, U5 D24V22F3, U6 D24V22F5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

Commit message: Added Stepper Motor Symbol, Erased Old MC
Katherine A. added in a symbol for a stepper motor and erased an outdated MC. Next on the agenda is updating the symbol library to be more accurate, adding in the motor driver, and adding all connections to the LattePanda
Parts:
- removed J1: LSS Conn, Connector_Molex:Molex_Mini-Fit_Jr_5566-04A_2x02_P4.20mm_Vertical, symbol Connector:Conn_01x04_Socket
- removed U2: Adafruit FeatherWing, Module:Adafruit_Feather, symbol Core_sym:Adafruit_Feather_ESP32_V2
- added M1: Stepper_Motor_bipolar, symbol Motor:Stepper_Motor_bipolar
Connections:
- net CS: no longer names the net of U1.7 (GPIO33/A5)
- net MISO: no longer names the net of U1.25 (GPIO19/MISO)
- net MOSI: no longer names the net of U1.30 (GPIO23/MOSI)
- net SCK: no longer names the net of U1.24 (GPIO18/SCK)
- net UART_MISO: no longer names the net of U1.21 (GPIO16/RX2)
- net UART_MOSI: no longer names the net of U1.22 (GPIO17/TX2)
- no-connect marks 56 -> 35
Other:
- note removed: "ESP32 FeatherWing"
